File: Kicad pcb/fotoaparat/fotoaparat.kicad_sch (KiCad schematic)
At the start: 66 parts, among them IC1 Lineární Regulátor, IC2 Lineární Regulátor Displaye, J1 USB Konektor, J2 SWD, J3 LCD konektor, J4 Baterie, J5 Sd Karta, J6 UART, J7 Kamera, U1 STM32L496RETx, U3 Nabíječka baterie, Y1 8mhz krystal

Commit message: Oprava chyb a volné konektory
Parts:
- added J8: Volné Piny, symbol Connector:Conn_01x12_Socket
- added R25: 1k, symbol Device:R
- added R26: 4.7k, symbol Device:R
Connections:
- net +3.3V: now also J5.4 (VDD1), U1.48 (VDDUSB), R25.1; no longer J5.3 (VSS1), J5.6 (VSS2)
- net +3.3VA: now also U1.13 (VDDA); no longer U1.48 (VDDUSB)
- net -BATT: now also J5.3 (VSS1), J5.6 (VSS2), R26.2; no longer J5.4 (VDD1)
- net csx: no longer J3.7, U1.9 (PC1)
- net pa2: now reaches U1.16 (PA2)
- net pa2: now also J8.4 (Pin_4)
- net pb0: now reaches U1.26 (PB0)
- net pb0: now also J8.2 (Pin_2)
- net pb1: now reaches U1.27 (PB1)
- net pb1: now also J8.1 (Pin_1)
- net pb12: now reaches U1.33 (PB12)
- net pb12: now also J8.10 (Pin_10)
- net pb14: now reaches U1.35 (PB14)
- net pb14: now also J8.11 (Pin_11)
- net pb15: now reaches U1.36 (PB15)
- net pb15: now also J8.12 (Pin_12)
- net pa8: now reaches U1.41 (PA8)
- net pa8: now also J8.5 (Pin_5)
- net pa9: now reaches U1.42 (PA9)
- net pa9: now also J8.6 (Pin_6)
- net pa10: now reaches U1.43 (PA10)
- net pa10: now also J8.7 (Pin_7)
- net pa15: now reaches U1.50 (PA15)
- net pa15: now also J8.3 (Pin_3)
- net pc10: now reaches U1.51 (PC10)
- net pc10: now also J8.8 (Pin_8)
- net pd2: now reaches U1.54 (PD2)
- net pd2: now also J8.9 (Pin_9)
- net Baterka Napětí: now reaches U1.8 (PC0)
- net Baterka Napětí: now also R25.2, R26.1
- new net sda: J3.7, U1.9 (PC1)
Other:
- moved on the sheet: C15
