File: Kicad pcb/fotoaparat/fotoaparat.kicad_pcb (KiCad board)
At the start: 2 copper layers, 27 parts, among them J1 USB Konektor, J2 SWD, J3 LCD konektor, J5 Sd Karta, J6 UART, J7 Kamera, U1 STM32L496RETx, U2 Regulator 3.3v, U3 MCP73833-FCI/UN, Y1 HC49S-8-30-50-70-30-ATF

Commit message: Baterie
Parts:
- added R6: MCU08050D1002BP500, 2012:RESC2012X55N, F.Cu at (121.5, 108.9)
- added R7: MCU08050D1002BP500, 2012:RESC2012X55N, F.Cu at (121.5, 112.0)
- added R8: MCU08050D1002BP500, 2012:RESC2012X55N, F.Cu at (121.5, 115.0)
- moved J5 9.75 mm to (137.5, 87.5)
- moved S2 5.98 mm to (167.4, 75.0)
- moved S1 0.50 mm to (170.8, 122.0)
Connections:
- J3 pad 1: unconnected-(J3-Pad1) -> Net-(J2-Pin_4)
- J3 pad 10: unconnected-(J3-Pad10) -> Net-(U1-PB1)
- J3 pad 11: unconnected-(J3-Pad11) -> Net-(J2-Pin_4)
- J3 pad 12: unconnected-(J3-Pad12) -> Net-(U1-PA6)
- J3 pad 14: unconnected-(J3-Pad14) -> Net-(J2-Pin_1)
- J3 pad 15: unconnected-(J3-Pad15) -> Net-(J2-Pin_4)
- J3 pad 2: unconnected-(J3-Pad2) -> Net-(J2-Pin_1)
- J3 pad 20: unconnected-(J3-Pad20) -> Net-(J2-Pin_4)
- J3 pad 3: unconnected-(J3-Pad3) -> Net-(J2-Pin_4)
- J3 pad 4: unconnected-(J3-Pad4) -> Net-(J2-Pin_4)
- J3 pad 5: unconnected-(J3-Pad5) -> Net-(J2-Pin_1)
- J3 pad 6: unconnected-(J3-Pad6) -> Net-(U1-PA11)
- J3 pad 7: unconnected-(J3-Pad7) -> Net-(U1-PA7)
- J3 pad 8: unconnected-(J3-Pad8) -> Net-(U1-PA1)
- J3 pad 9: unconnected-(J3-Pad9) -> Net-(U1-PB0)
- J3 pad S1: Net-(J3-SHIELD-PadS1) -> Net-(J2-Pin_4)
- J3 pad S2: Net-(J3-SHIELD-PadS1) -> Net-(J2-Pin_4)
- J3 pad S3: Net-(J3-SHIELD-PadS1) -> Net-(J2-Pin_4)
- J3 pad S4: Net-(J3-SHIELD-PadS1) -> Net-(J2-Pin_4)
- J5 pad 1: unconnected-(J5-CD/DAT3-Pad1) -> Net-(J5-CD/DAT3)
- J5 pad 12: unconnected-(J5-GND-Pad12) -> Net-(J2-Pin_4)
- J5 pad 13: unconnected-(J5-GND-Pad13) -> Net-(J2-Pin_4)
- J5 pad 14: unconnected-(J5-GND-Pad14) -> Net-(J2-Pin_4)
- J5 pad 15: unconnected-(J5-GND-Pad15) -> Net-(J2-Pin_4)
- J5 pad 2: unconnected-(J5-CMD-Pad2) -> Net-(J5-CMD)
- J5 pad 3: unconnected-(J5-VSS1-Pad3) -> Net-(J2-Pin_4)
- J5 pad 4: unconnected-(J5-VDD1-Pad4) -> Net-(J2-Pin_1)
- J5 pad 5: unconnected-(J5-CLK-Pad5) -> Net-(J5-CLK)
- J5 pad 7: unconnected-(J5-DAT0-Pad7) -> Net-(J5-DAT0)
- R1 pad 2: Net-(S5-COM_1) -> Net-(J5-CD/DAT3)
- S1 pad MH1: unconnected-(S1-PadMH1) -> Net-(J2-Pin_4)
- S1 pad MH2: unconnected-(S1-PadMH2) -> Net-(J2-Pin_4)
- S1 pad MH3: unconnected-(S1-PadMH3) -> Net-(J2-Pin_4)
- S1 pad MH4: unconnected-(S1-PadMH4) -> Net-(J2-Pin_4)
- S5 pad A1: Net-(S5-COM_1) -> Net-(J5-CD/DAT3)
- U1 pad 10: Net-(J7-Pin_21) -> Net-(J5-DAT0)
- U1 pad 15: unconnected-(U1-PA1-Pad15) -> Net-(U1-PA1)
- U1 pad 22: unconnected-(U1-PA6-Pad22) -> Net-(U1-PA6)
- U1 pad 23: unconnected-(U1-PA7-Pad23) -> Net-(U1-PA7)
- U1 pad 26: unconnected-(U1-PB0-Pad26) -> Net-(U1-PB0)
- U1 pad 27: unconnected-(U1-PB1-Pad27) -> Net-(U1-PB1)
- U1 pad 29: unconnected-(U1-PB10-Pad29) -> Net-(J5-CLK)
- U1 pad 33: unconnected-(U1-PB12-Pad33) -> Net-(J5-CD/DAT3)
- U1 pad 36: unconnected-(U1-PB15-Pad36) -> Net-(J5-CMD)
- U1 pad 44: unconnected-(U1-PA11-Pad44) -> Net-(U1-PA11)
- U1 pad 60: Net-(S5-COM_1) -> Net-(J5-CD/DAT3)
- U1 pad 9: unconnected-(U1-PC1-Pad9) -> Net-(J7-Pin_21)
- U3 pad 1: unconnected-(U3-VDD-Pad1) -> Net-(J4-Pin_1)
- U3 pad 10: unconnected-(U3-VBAT-Pad10) -> Net-(J4-Pin_2)

Commit message: Přepojení součástek
vypadá to trochu lépe
Parts:
- added C10: 100n, Capacitor_SMD:C_0603_1608Metric_Pad1.08x0.95mm_HandSolder, F.Cu at (114.1, 127.5)
- added C11: 100n, Capacitor_SMD:C_0603_1608Metric_Pad1.08x0.95mm_HandSolder, F.Cu at (114.1, 130.0)
- added C12: 100n, Capacitor_SMD:C_0603_1608Metric_Pad1.08x0.95mm_HandSolder, F.Cu at (114.1, 132.5)
- added C14: 10n, Capacitor_SMD:C_0603_1608Metric_Pad1.08x0.95mm_HandSolder, F.Cu at (114.1, 135.0)
- added C17: 30p, Capacitor_SMD:C_0201_0603Metric_Pad0.64x0.40mm_HandSolder, F.Cu at (117.7, 124.6)
- added C18: 30p, Capacitor_SMD:C_0201_0603Metric_Pad0.64x0.40mm_HandSolder, F.Cu at (117.7, 126.3)
- added C9: 100n, Capacitor_SMD:C_0603_1608Metric_Pad1.08x0.95mm_HandSolder, F.Cu at (114.1, 125.0)
- R1, R2, R3: value MCU08050D1002BP500 -> 1.5k
- S2: value MC32829 -> tlačítko doleva
- S3: value MC32829 -> prostřední tlačítko
- S4: value MC32829 -> tlačítko doprava
- S5: value CFS-0201MB -> spínač
- Y1: value HC49S-8-30-50-70-30-ATF -> 8mhz krystal
- moved J3 7.75 mm to (178.6, 106.8), turned to 90 degrees
Connections:
- net Net-(J7-Pin_10) renamed /d4
- net Net-(J7-Pin_11) renamed /d3
- net Net-(J7-Pin_12) renamed /d2
- net Net-(J7-Pin_14) renamed /d0
- net Net-(J7-Pin_5) renamed /vsync
- net Net-(J7-Pin_6) renamed /href
- net Net-(J7-Pin_7) renamed /d7
- net Net-(J7-Pin_8) renamed /d6
- net Net-(J7-Pin_9) renamed /d5
- J1 pad 1: unconnected-(J1-VBUS-Pad1) -> VBUS
- J1 pad 2: unconnected-(J1-D--Pad2) -> /data -
- J1 pad 3: unconnected-(J1-D+-Pad3) -> /data +
- J1 pad 5: Net-(J1-GND) -> GND
- J2 pad 1: Net-(J2-Pin_1) -> +3.3V
- J2 pad 2: Net-(J2-Pin_2) -> /swdio
- J2 pad 3: Net-(J2-Pin_3) -> /swclk
- J2 pad 4: Net-(J2-Pin_4) -> GND
- J3 pad 1: Net-(J2-Pin_4) -> GND
- J3 pad 10: Net-(U1-PB1) -> unconnected-(J3-Pad10)
- J3 pad 11: Net-(J2-Pin_4) -> GND
- J3 pad 12: Net-(U1-PA6) -> /sdo
- J3 pad 14: Net-(J2-Pin_1) -> Net-(J3-Pad14)
- J3 pad 15: Net-(J2-Pin_4) -> GND
- J3 pad 2: Net-(J2-Pin_1) -> +3.3V
- J3 pad 20: Net-(J2-Pin_4) -> GND
- J3 pad 3: Net-(J2-Pin_4) -> GND
- J3 pad 4: Net-(J2-Pin_4) -> GND
- J3 pad 5: Net-(J2-Pin_1) -> +3.3V
- J3 pad 6: Net-(U1-PA11) -> unconnected-(J3-Pad6)
- J3 pad 7: Net-(U1-PA7) -> /sda
- J3 pad 8: Net-(U1-PA1) -> /scl
- J3 pad 9: Net-(U1-PB0) -> unconnected-(J3-Pad9)
- J3 pad S1: Net-(J2-Pin_4) -> unconnected-(J3-SHIELD-PadS1)_1
- J3 pad S2: Net-(J2-Pin_4) -> unconnected-(J3-SHIELD-PadS1)_3
- J3 pad S3: Net-(J2-Pin_4) -> unconnected-(J3-SHIELD-PadS1)_2
- J3 pad S4: Net-(J2-Pin_4) -> unconnected-(J3-SHIELD-PadS1)
- J5 pad 1: Net-(J5-CD/DAT3) -> /sd cs
- J5 pad 12: Net-(J2-Pin_4) -> unconnected-(J5-GND-Pad12)
- J5 pad 13: Net-(J2-Pin_4) -> unconnected-(J5-GND-Pad13)
- J5 pad 14: Net-(J2-Pin_4) -> unconnected-(J5-GND-Pad14)
- J5 pad 15: Net-(J2-Pin_4) -> unconnected-(J5-GND-Pad15)
- J5 pad 2: Net-(J5-CMD) -> /sd mosi
- J5 pad 3: Net-(J2-Pin_4) -> +3.3V
- J5 pad 4: Net-(J2-Pin_1) -> GND
- J5 pad 5: Net-(J5-CLK) -> /sd clk
- J5 pad 6: unconnected-(J5-VSS2-Pad6) -> +3.3V
- J5 pad 7: Net-(J5-DAT0) -> /sd miso
- J6 pad 1: Net-(J6-Pin_1) -> /uart tx
- J6 pad 2: Net-(J6-Pin_2) -> /uart rx
- J7 pad 1: Net-(J2-Pin_1) -> +3.3V
- J7 pad 13: Net-(J7-Pin_13) -> /d1
- J7 pad 15: Net-(J2-Pin_1) -> +3.3V
- J7 pad 18: Net-(J7-Pin_18) -> /rck
- J7 pad 19: Net-(J7-Pin_19) -> /wr
- J7 pad 2: Net-(J2-Pin_4) -> GND
- J7 pad 20: Net-(J2-Pin_4) -> GND
- J7 pad 21: Net-(J7-Pin_21) -> /wrst
- J7 pad 22: Net-(J7-Pin_22) -> /rrst
- J7 pad 3: Net-(J7-Pin_3) -> /scl
- J7 pad 4: Net-(J7-Pin_4) -> /sda
- R1 pad 1: Net-(J2-Pin_4) -> +3.3V
- R1 pad 2: Net-(J5-CD/DAT3) -> /sw3
- R2 pad 1: Net-(J2-Pin_1) -> +3.3V
- R2 pad 2: Net-(S5-COM_2) -> /sw2
- R3 pad 1: Net-(U1-PA8) -> +3.3V
- R3 pad 2: Net-(J2-Pin_4) -> /sw1
- S1 pad MH1: Net-(J2-Pin_4) -> unconnected-(S1-PadMH1)
- S1 pad MH2: Net-(J2-Pin_4) -> unconnected-(S1-PadMH2)
- S1 pad MH3: Net-(J2-Pin_4) -> unconnected-(S1-PadMH3)
- S1 pad MH4: Net-(J2-Pin_4) -> unconnected-(S1-PadMH4)
- S2 pad 1: Net-(J2-Pin_1) -> unconnected-(S2-Pad1)
- S2 pad 2: Net-(U1-PA8) -> unconnected-(S2-Pad2)
- S2 pad 3: unconnected-(S2-Pad3) -> GND
- S2 pad 4: unconnected-(S2-Pad4) -> /sw1
- S3 pad 1: Net-(J2-Pin_1) -> unconnected-(S3-Pad1)
- S3 pad 2: Net-(U1-PA9) -> unconnected-(S3-Pad2)
- S3 pad 3: unconnected-(S3-Pad3) -> GND
- S3 pad 4: unconnected-(S3-Pad4) -> /sw2
- S4 pad 1: Net-(J2-Pin_1) -> unconnected-(S4-Pad1)
- S4 pad 2: Net-(U1-PA5) -> unconnected-(S4-Pad2)
- S4 pad 3: unconnected-(S4-Pad3) -> GND
- S4 pad 4: unconnected-(S4-Pad4) -> /sw3
- S5 pad A1: Net-(J5-CD/DAT3) -> /Reset
- S5 pad A2: Net-(S5-COM_2) -> +3.3V
- S5 pad B1: Net-(J2-Pin_1) -> GND
- S5 pad B2: Net-(J2-Pin_4) -> /boot0
- U1 pad 1: unconnected-(U1-VBAT-Pad1) -> +3.3V
- U1 pad 10: Net-(J5-DAT0) -> /sdo
- U1 pad 11: Net-(J7-Pin_19) -> /sw1
- U1 pad 12: Net-(J2-Pin_4) -> GND
- U1 pad 13: Net-(J2-Pin_1) -> unconnected-(U1-VDDA-Pad13)
- U1 pad 14: unconnected-(U1-PA0-Pad14) -> /uart tx
- U1 pad 15: Net-(U1-PA1) -> /uart rx
- U1 pad 16: Net-(J6-Pin_1) -> unconnected-(U1-PA2-Pad16)
- U1 pad 17: Net-(J6-Pin_2) -> /sd cs
- U1 pad 18: Net-(J2-Pin_4) -> GND
- U1 pad 19: Net-(J2-Pin_1) -> +3.3V
- U1 pad 2: unconnected-(U1-PC13-Pad2) -> /rrst
- U1 pad 21: Net-(U1-PA5) -> /sd clk
- U1 pad 22: Net-(U1-PA6) -> /wr
- U1 pad 23: Net-(U1-PA7) -> /sd mosi
- U1 pad 24: Net-(J7-Pin_22) -> /sw2
- U1 pad 25: Net-(J7-Pin_18) -> /sw3
- U1 pad 26: Net-(U1-PB0) -> unconnected-(U1-PB0-Pad26)
- U1 pad 27: Net-(U1-PB1) -> unconnected-(U1-PB1-Pad27)
- U1 pad 29: Net-(J5-CLK) -> /scl
- U1 pad 3: unconnected-(U1-PC14-Pad3) -> /wrst
- U1 pad 30: unconnected-(U1-PB11-Pad30) -> /sda
- U1 pad 31: Net-(J2-Pin_4) -> GND
- U1 pad 32: Net-(J2-Pin_1) -> +3.3V
- U1 pad 33: Net-(J5-CD/DAT3) -> unconnected-(U1-PB12-Pad33)
- U1 pad 34: Net-(J7-Pin_3) -> /scl
- U1 pad 35: Net-(J7-Pin_4) -> unconnected-(U1-PB14-Pad35)
- U1 pad 36: Net-(J5-CMD) -> unconnected-(U1-PB15-Pad36)
- U1 pad 38: unconnected-(U1-PC7-Pad38) -> /d1
- U1 pad 41: Net-(U1-PA8) -> unconnected-(U1-PA8-Pad41)
- U1 pad 42: Net-(U1-PA9) -> unconnected-(U1-PA9-Pad42)
- U1 pad 43: Net-(J7-Pin_13) -> unconnected-(U1-PA10-Pad43)
- U1 pad 44: Net-(U1-PA11) -> /data -
- U1 pad 45: unconnected-(U1-PA12-Pad45) -> /data +
- U1 pad 46: Net-(J2-Pin_3) -> /swdio
- U1 pad 47: Net-(J2-Pin_4) -> GND
- U1 pad 48: unconnected-(U1-VDDUSB-Pad48) -> +3.3VA
- U1 pad 49: Net-(J2-Pin_2) -> /swclk
- U1 pad 5: Net-(U1-PH0) -> /osc in
- U1 pad 53: unconnected-(U1-PC12-Pad53) -> /rck
- U1 pad 56: unconnected-(U1-PB4-Pad56) -> /sd miso
- U1 pad 6: Net-(U1-PH1) -> /osc out
- U1 pad 60: Net-(J5-CD/DAT3) -> /boot0
- U1 pad 63: Net-(J2-Pin_4) -> GND
- U1 pad 64: Net-(J2-Pin_1) -> +3.3V
- U1 pad 7: Net-(S5-COM_2) -> /Reset
- U1 pad 9: Net-(J7-Pin_21) -> /sda
- U3 pad 1: Net-(J4-Pin_1) -> unconnected-(U3-VDD-Pad1)
- U3 pad 10: Net-(J4-Pin_2) -> unconnected-(U3-VBAT-Pad10)
- U3 pad 5: Net-(J1-GND) -> unconnected-(U3-VSS-Pad5)
- Y1 pad 1: Net-(U1-PH1) -> /osc in
- Y1 pad 2: Net-(U1-PH0) -> /osc out

Commit message: Regulátory
Parts:
- removed U2: Regulator 3.3v, MPQ:QFN-3x4_MPQ4432_MNP
- added C13: 1u, Capacitor_SMD:C_0805_2012Metric_Pad1.18x1.45mm_HandSolder, F.Cu at (147.5, 103.1)
- added C15: 1u, Capacitor_SMD:C_0805_2012Metric_Pad1.18x1.45mm_HandSolder, F.Cu at (147.5, 109.1)
- added C16: 1u, Capacitor_SMD:C_0805_2012Metric_Pad1.18x1.45mm_HandSolder, F.Cu at (152.3, 97.0)
- added C19: 1u, Capacitor_SMD:C_0805_2012Metric_Pad1.18x1.45mm_HandSolder, F.Cu at (152.3, 106.1)
- added C20: 1u, Capacitor_SMD:C_0805_2012Metric_Pad1.18x1.45mm_HandSolder, F.Cu at (152.3, 109.1)
- added C8: 1u, Capacitor_SMD:C_0805_2012Metric_Pad1.18x1.45mm_HandSolder, F.Cu at (142.7, 103.1)
- added D1: LED, LED_SMD:LED_0805_2012Metric_Pad1.15x1.40mm_HandSolder, F.Cu at (172.0, 103.4)
- added D2: LED, LED_SMD:LED_0805_2012Metric_Pad1.15x1.40mm_HandSolder, F.Cu at (172.0, 106.5)
- added D3: LED, LED_SMD:LED_0805_2012Metric_Pad1.15x1.40mm_HandSolder, F.Cu at (172.0, 109.5)
- added FB1: 120R, Inductor_SMD:L_0805_2012Metric_Pad1.05x1.20mm_HandSolder, F.Cu at (161.8, 91.2)
- added IC1: Lineární Regulátor, Package_TO_SOT_SMD:TSOT-23-5_HandSoldering, F.Cu at (167.8, 114.9)
- added IC2: Lineární Regulátor Displaye, Package_TO_SOT_SMD:TSOT-23-5_HandSoldering, F.Cu at (167.8, 119.4)
- added J4: Baterie, Connector_PinSocket_2.54mm:PinSocket_1x02_P2.54mm_Horizontal, F.Cu at (172.6, 68.6)
- added R10: 4.7k, Resistor_SMD:R_0805_2012Metric_Pad1.20x1.40mm_HandSolder, F.Cu at (142.6, 120.9)
- added R11: 4.7k, Resistor_SMD:R_0805_2012Metric_Pad1.20x1.40mm_HandSolder, F.Cu at (142.6, 123.9)
- added R12: 4.7k, Resistor_SMD:R_0805_2012Metric_Pad1.20x1.40mm_HandSolder, F.Cu at (142.6, 126.8)
- added R13: 4.7k, Resistor_SMD:R_0805_2012Metric_Pad1.20x1.40mm_HandSolder, F.Cu at (147.4, 112.1)
- added R14: 4.7k, Resistor_SMD:R_0805_2012Metric_Pad1.20x1.40mm_HandSolder, F.Cu at (147.4, 115.0)
- added R15: 4.7k, Resistor_SMD:R_0805_2012Metric_Pad1.20x1.40mm_HandSolder, F.Cu at (147.4, 118.0)
- added R16: 4.7k, Resistor_SMD:R_0805_2012Metric_Pad1.20x1.40mm_HandSolder, F.Cu at (147.4, 120.9)
- added R17: 4.7k, Resistor_SMD:R_0805_2012Metric_Pad1.20x1.40mm_HandSolder, F.Cu at (147.4, 123.9)
- added R18: 4.7k, Resistor_SMD:R_0805_2012Metric_Pad1.20x1.40mm_HandSolder, F.Cu at (147.4, 126.8)
- added R19: 4.7k, Resistor_SMD:R_0805_2012Metric_Pad1.20x1.40mm_HandSolder, F.Cu at (152.1, 112.1)
- added R20: 4.7k, Resistor_SMD:R_0805_2012Metric_Pad1.20x1.40mm_HandSolder, F.Cu at (152.1, 115.0)
- added R21: 4.7k, Resistor_SMD:R_0805_2012Metric_Pad1.20x1.40mm_HandSolder, F.Cu at (152.1, 118.0)
- added R22: 4.7k, Resistor_SMD:R_0805_2012Metric_Pad1.20x1.40mm_HandSolder, F.Cu at (152.1, 120.9)
- added R23: 4.7k, Resistor_SMD:R_0805_2012Metric_Pad1.20x1.40mm_HandSolder, F.Cu at (152.1, 123.9)
- added R24: 4.7k, Resistor_SMD:R_0805_2012Metric_Pad1.20x1.40mm_HandSolder, F.Cu at (152.1, 126.8)
- added R9: 4.7k, Resistor_SMD:R_0805_2012Metric_Pad1.20x1.40mm_HandSolder, F.Cu at (142.6, 118.0)
- added TH1: 10k, Connector_PinSocket_2.54mm:PinSocket_1x02_P2.54mm_Horizontal, F.Cu at (172.6, 75.8)
- C1, C2, C3, C4: value MC0603B104K250CT -> 1u; footprint mc06:CAPC1608X87N -> Capacitor_SMD:C_0805_2012Metric_Pad1.18x1.45mm_HandSolder
- C10, C11, C12, C9: footprint Capacitor_SMD:C_0603_1608Metric_Pad1.08x0.95mm_HandSolder -> Capacitor_SMD:C_0805_2012Metric_Pad1.18x1.45mm_HandSolder
- C14: value 10n -> 100n; footprint Capacitor_SMD:C_0603_1608Metric_Pad1.08x0.95mm_HandSolder -> Capacitor_SMD:C_0805_2012Metric_Pad1.18x1.45mm_HandSolder
- C17, C18: footprint Capacitor_SMD:C_0201_0603Metric_Pad0.64x0.40mm_HandSolder -> Capacitor_SMD:C_0805_2012Metric_Pad1.18x1.45mm_HandSolder
- C5: value MC0805B105K160CT -> 1u; footprint mc08:CAPC2012X135N -> Capacitor_SMD:C_0805_2012Metric_Pad1.18x1.45mm_HandSolder
- C6, C7: value GRM0335C1H300GA01D -> 1u; footprint grm033:GRM033D70J224ME01D -> Capacitor_SMD:C_0805_2012Metric_Pad1.18x1.45mm_HandSolder
- J2: footprint Connector_PinSocket_2.54mm:PinSocket_1x04_P2.54mm_Vertical -> Connector_PinHeader_2.54mm:PinHeader_1x04_P2.54mm_Vertical
- J6: footprint Connector_PinSocket_2.54mm:PinSocket_1x02_P2.54mm_Vertical -> Connector_PinHeader_2.54mm:PinHeader_1x02_P2.54mm_Vertical
- J7: footprint Connector_PinHeader_2.54mm:PinHeader_2x11_P2.54mm_Vertical -> Connector_PinSocket_2.54mm:PinSocket_2x11_P2.54mm_Vertical
- R1, R2, R3: value 1.5k -> 4.7k; footprint 2012:RESC2012X55N -> Resistor_SMD:R_0805_2012Metric_Pad1.20x1.40mm_HandSolder
- R4, R5, R6, R7: value MCU08050D1002BP500 -> 1k; footprint 2012:RESC2012X55N -> Resistor_SMD:R_0805_2012Metric_Pad1.20x1.40mm_HandSolder
- R8: value MCU08050D1002BP500 -> 2; footprint 2012:RESC2012X55N -> Resistor_SMD:R_0805_2012Metric_Pad1.20x1.40mm_HandSolder
- S1: value MFS201N-24-Z -> Zapínací spínač
- U3: value MCP73833-FCI/UN -> Nabíječka baterie
- moved J7 67.6 mm to (121.5, 97.9)
- moved R3 55.2 mm to (137.9, 118.0)
- moved R4 55.1 mm to (137.9, 120.9)
- moved R5 55.0 mm to (137.9, 123.9)
- moved J6 52.6 mm to (173.2, 83.1)
- moved C11 46.9 mm to (147.5, 97.0)
- moved C12 46.5 mm to (147.5, 100.0)
- moved S2 45.4 mm to (129.6, 100.2)
- moved C14 44.2 mm to (147.5, 106.1)
- moved S3 42.4 mm to (129.6, 109.5)
- moved S4 42.4 mm to (129.6, 118.8)
- moved C17 42.4 mm to (152.3, 100.0)
- moved U1 42.2 mm to (154.3, 73.6)
- moved C18 41.7 mm to (152.3, 103.1)
- moved J1 41.1 mm to (165.1, 85.6)
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Connections:
- net /data + renamed /USB_D+
- net /data - renamed /USB_D-
- C1 pad 1: Net-(J2-Pin_4) -> VBUS
- C1 pad 2: Net-(J2-Pin_1) -> -BATT
- C10 pad 1: GND -> -BATT
- C11 pad 1: GND -> -BATT
- C12 pad 1: GND -> -BATT
- C14 pad 2: GND -> -BATT
- C17 pad 1: GND -> -BATT
- C18 pad 1: GND -> -BATT
- C2 pad 1: Net-(J2-Pin_4) -> +BATT
- C2 pad 2: Net-(J2-Pin_1) -> -BATT
- C3 pad 1: Net-(J2-Pin_4) -> +BATT
- C3 pad 2: Net-(J2-Pin_1) -> -BATT
- C4 pad 1: Net-(J2-Pin_4) -> -BATT
- C4 pad 2: Net-(J2-Pin_1) -> +3.3V
- C5 pad 1: Net-(J2-Pin_4) -> +BATT
- C5 pad 2: Net-(J2-Pin_1) -> -BATT
- C6 pad 1: Net-(U1-PH1) -> -BATT
- C6 pad 2: Net-(J2-Pin_4) -> +3.3V LCD
- C7 pad 1: Net-(U1-PH0) -> -BATT
- C7 pad 2: Net-(J2-Pin_4) -> +3.3V
- C9 pad 1: GND -> -BATT
- J1 pad 5: GND -> -BATT
- J2 pad 4: GND -> -BATT
- J3 pad 1: GND -> -BATT
- J3 pad 10: unconnected-(J3-Pad10) -> /wrx d/cx
- J3 pad 11: GND -> -BATT
- J3 pad 15: GND -> -BATT
- J3 pad 2: +3.3V -> Net-(J3-Pad2)
- J3 pad 20: GND -> -BATT
- J3 pad 3: GND -> -BATT
- J3 pad 4: GND -> -BATT
- J3 pad 5: +3.3V -> +3.3V LCD
- J3 pad 6: unconnected-(J3-Pad6) -> /rst
- J3 pad 7: /sda -> /csx
- J3 pad 9: unconnected-(J3-Pad9) -> /csx
- J5 pad 4: GND -> -BATT
- J7 pad 2: GND -> -BATT
- J7 pad 20: GND -> -BATT
- J7 pad 4: /sda -> /sdo
- R4 pad 2: Net-(J2-Pin_4) -> Net-(U3-STAT1)
- R5 pad 2: Net-(J2-Pin_4) -> Net-(U3-STAT2)
- R6 pad 1: Net-(J2-Pin_1) -> /Indikátor Nabíjení
- R6 pad 2: Net-(J5-CD/DAT3) -> Net-(U3-*PG)
- R7 pad 1: Net-(J2-Pin_1) -> Net-(U3-PROG)
- R7 pad 2: Net-(J5-DAT0) -> -BATT
- R8 pad 1: Net-(J2-Pin_1) -> +3.3V LCD
- R8 pad 2: Net-(J5-CMD) -> Net-(J3-Pad2)
- S1 pad 2: unconnected-(S1-COM_1-Pad2) -> +BATT
- S1 pad 3: unconnected-(S1-NO_1-Pad3) -> Net-(IC1-EN)
- S1 pad 5: unconnected-(S1-COM_2-Pad5) -> /Backlight Regulátor
- S1 pad 6: unconnected-(S1-NO_2-Pad6) -> Net-(IC2-EN)
- S2 pad 3: GND -> -BATT
- S3 pad 3: GND -> -BATT
- S4 pad 3: GND -> -BATT
- S5 pad B1: GND -> -BATT
- U1 pad 12: GND -> -BATT
- U1 pad 18: GND -> -BATT
- U1 pad 28: unconnected-(U1-PB2-Pad28) -> /rst
- U1 pad 30: /sda -> /sdo
- U1 pad 31: GND -> -BATT
- U1 pad 4: unconnected-(U1-PC15-Pad4) -> /Backlight Regulátor
- U1 pad 47: GND -> -BATT
- U1 pad 55: unconnected-(U1-PB3-Pad55) -> /csx
- U1 pad 57: unconnected-(U1-PB5-Pad57) -> /wrx d/cx
- U1 pad 63: GND -> -BATT
- U1 pad 9: /sda -> /csx
- U3 pad 1: unconnected-(U3-VDD-Pad1) -> VBUS
- U3 pad 10: unconnected-(U3-VBAT-Pad10) -> +BATT
- U3 pad 2: unconnected-(U3-VDD-Pad2) -> VBUS
- U3 pad 3: unconnected-(U3-STAT1-Pad3) -> Net-(U3-STAT1)
- U3 pad 4: unconnected-(U3-STAT2-Pad4) -> Net-(U3-STAT2)
- U3 pad 5: unconnected-(U3-VSS-Pad5) -> -BATT
- U3 pad 6: unconnected-(U3-PROG-Pad6) -> Net-(U3-PROG)
- U3 pad 7: unconnected-(U3-*PG-Pad7) -> Net-(U3-*PG)
- U3 pad 8: unconnected-(U3-THERM-Pad8) -> Net-(U3-THERM)
- U3 pad 9: unconnected-(U3-VBAT-Pad9) -> +BATT

Commit message: Začátek návrhu pcb desky
Parts:
- removed IC2: Lineární Regulátor Displaye, Package_TO_SOT_SMD:TSOT-23-5_HandSoldering
- removed U3: Nabíječka baterie, MCP:MSOP10_MC_MCH
- added BZ1: Buzzer, Inductor_SMD:L_SXN_SMDRI73, F.Cu at (84.0, 97.0)
- added C21: 100n, Capacitor_SMD:C_0805_2012Metric_Pad1.18x1.45mm_HandSolder, F.Cu at (85.0, 88.4)
- added IC3: Lineární Regulátor Displaye, Package_TO_SOT_SMD:TSOT-23-5_HandSoldering, F.Cu at (102.0, 117.0)
- added J9: Conn_01x11_Socket, Connector_PinSocket_2.54mm:PinSocket_1x11_P2.54mm_Horizontal, F.Cu at (120.7, 64.4)
- added R25: 1k, Resistor_SMD:R_0805_2012Metric_Pad1.20x1.40mm_HandSolder, F.Cu at (121.0, 111.0)
- added R26: 4.7k, Resistor_SMD:R_0805_2012Metric_Pad1.20x1.40mm_HandSolder, F.Cu at (121.0, 115.0)
- added U2: MCP73833-FCI/UN, MCP:MSOP10_MC_MCH, F.Cu at (116.0, 95.0)
- J5: value Sd Karta -> GSD090012SEU
- J7: moved to B.Cu
- S5: footprint cfs:CFS0201MB -> cfs201mb:CFS0201MB
- moved J3 133.8 mm to (31.6, 80.2), turned to -90 degrees
- moved R13 127.9 mm to (23.0, 82.0), turned to -90 degrees
- moved J6 122.2 mm to (51.0, 86.0)
- moved R9 115.9 mm to (38.0, 68.0), turned to -90 degrees
- moved R8 114.2 mm to (31.0, 91.0), turned to 180 degrees
- moved S5 111.0 mm to (58.0, 75.0)
- moved R10 108.4 mm to (48.0, 68.0), turned to -90 degrees
- moved R12 103.6 mm to (58.0, 67.0)
- moved R21 102.7 mm to (52.0, 95.0), turned to -90 degrees
- moved R22 102.5 mm to (52.0, 99.0), turned to -90 degrees
- moved R23 102.3 mm to (52.0, 103.0), turned to -90 degrees
- moved R11 94.0 mm to (58.0, 83.0), turned to 180 degrees
- moved R18 89.6 mm to (64.0, 94.0), turned to -90 degrees
- moved C17 89.4 mm to (68.0, 70.4), turned to 180 degrees
- moved R19 89.2 mm to (64.0, 98.0), turned to -90 degrees
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Connections:
- net Net-(J3-Pad14) renamed /im3
- net Net-(J3-Pad2) renamed /Vled+
- C1 pad 2: -BATT -> GND
- C10 pad 1: -BATT -> GND
- C11 pad 1: -BATT -> GND
- C12 pad 1: -BATT -> GND
- C13 pad 1: -BATT -> GND
- C14 pad 2: -BATT -> GND
- C15 pad 2: -BATT -> GND
- C16 pad 2: -BATT -> GND
- C17 pad 1: -BATT -> GND
- C18 pad 1: -BATT -> GND
- C19 pad 1: -BATT -> GND
- C2 pad 2: -BATT -> GND
- C20 pad 1: -BATT -> GND
- C3 pad 2: -BATT -> GND
- C4 pad 1: -BATT -> GND
- C5 pad 2: -BATT -> GND
- C6 pad 1: -BATT -> GND
- C7 pad 1: -BATT -> GND
- C8 pad 1: -BATT -> GND
- C9 pad 1: -BATT -> GND
- IC1 pad 2: -BATT -> GND
- J1 pad 5: -BATT -> GND
- J2 pad 4: -BATT -> GND
- J3 pad 1: -BATT -> GND
- J3 pad 11: -BATT -> GND
- J3 pad 15: -BATT -> GND
- J3 pad 20: -BATT -> GND
- J3 pad 3: -BATT -> GND
- J3 pad 4: -BATT -> GND
- J3 pad 7: /csx -> /sda
- J4 pad 2: -BATT -> GND
- J5 pad 3: +3.3V -> GND
- J5 pad 4: -BATT -> +3.3V
- J5 pad 6: +3.3V -> GND
- J7 pad 2: -BATT -> GND
- J7 pad 20: -BATT -> GND
- J7 pad 3: /scl -> /I2C_SCL
- J7 pad 4: /sdo -> /I2C_SDA
- R10 pad 2: /sdo -> /I2C_SDA
- R12 pad 1: -BATT -> GND
- R14 pad 1: -BATT -> GND
- R24 pad 1: -BATT -> GND
- R7 pad 2: -BATT -> GND
- R9 pad 2: /scl -> /I2C_SCL
- S2 pad 3: -BATT -> GND
- S3 pad 3: -BATT -> GND
- S4 pad 3: -BATT -> GND
- S5 pad B1: -BATT -> GND
- TH1 pad 2: -BATT -> GND
- U1 pad 12: -BATT -> GND
- U1 pad 13: unconnected-(U1-VDDA-Pad13) -> +3.3VA
- U1 pad 16: unconnected-(U1-PA2-Pad16) -> /pa2
- U1 pad 18: -BATT -> GND
- U1 pad 26: unconnected-(U1-PB0-Pad26) -> /pb0
- U1 pad 27: unconnected-(U1-PB1-Pad27) -> /pb1
- U1 pad 29: /scl -> /I2C_SCL
- U1 pad 30: /sdo -> /I2C_SDA
- U1 pad 31: -BATT -> GND
- U1 pad 33: unconnected-(U1-PB12-Pad33) -> /pb12
- U1 pad 35: unconnected-(U1-PB14-Pad35) -> /pb14
- U1 pad 36: unconnected-(U1-PB15-Pad36) -> /buzzer
- U1 pad 41: unconnected-(U1-PA8-Pad41) -> /pa8
- U1 pad 42: unconnected-(U1-PA9-Pad42) -> /pa9
- U1 pad 43: unconnected-(U1-PA10-Pad43) -> /pa10
- U1 pad 47: -BATT -> GND
- U1 pad 48: +3.3VA -> +3.3V
- U1 pad 50: unconnected-(U1-PA15-Pad50) -> /pa15
- U1 pad 51: unconnected-(U1-PC10-Pad51) -> /pc10
- U1 pad 54: unconnected-(U1-PD2-Pad54) -> /pd2
- U1 pad 63: -BATT -> GND
- U1 pad 8: unconnected-(U1-PC0-Pad8) -> /Baterka Napětí
- U1 pad 9: /csx -> /sda

Commit message: Outline desky
Parts:
- added H1: MountingHole, MountingHole:MountingHole_3.2mm_M3, F.Cu at (196.4, 139.4)
- added H2: MountingHole, MountingHole:MountingHole_3.2mm_M3, F.Cu at (86.4, 139.4)
- added H3: MountingHole, MountingHole:MountingHole_3.2mm_M3, F.Cu at (86.4, 64.4)
- added H4: MountingHole, MountingHole:MountingHole_3.2mm_M3, F.Cu at (196.4, 64.4)
- Free Pins: renamed from J9
- SD CARD: renamed from J5
- UART TX: renamed from J6
- moved USB 76.5 mm to (199.9, 82.1)
- moved R21 72.6 mm to (123.0, 110.0), turned to 180 degrees
- moved C3 71.6 mm to (176.5, 116.4)
- moved R25 71.5 mm to (192.4, 116.0)
- moved R26 71.5 mm to (192.4, 120.0)
- moved C9 71.5 mm to (149.4, 93.4)
- moved Free Pins 71.5 mm to (192.0, 68.8)
- moved R10 71.5 mm to (119.4, 72.4)
- moved R13 71.5 mm to (94.4, 86.4)
- moved R8 71.5 mm to (102.4, 95.4)
- moved R9 71.5 mm to (109.4, 72.4)
- moved UART TX 71.5 mm to (122.4, 90.4)
- moved +BATT 71.5 mm to (188.8, 114.1)
- moved BZ1 71.5 mm to (155.4, 101.4)
- moved C1 71.5 mm to (190.4, 99.4)
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- renumbered J4 to +BATT, J7 to CAMERA, J3 to LCD, J2 to SWD, J1 to USB
Routing:
- net +3.3V: track 0.00 -> 7.57 mm
- net GND: track 0.00 -> 6.50 mm
- added copper zone on B.Cu, net GND
Other:
- board outline added: 120 x 85 mm

Commit message: První pcb spoje
Routing:
- net GND: track 6.50 -> 54.4 mm, vias 0 -> 16
- net /sw3: track 0.00 -> 11.5 mm
- net /sw1: track 0.00 -> 11.1 mm
- net /sw2: track 0.00 -> 11.0 mm
- net +3.3V: track 7.57 -> 18.3 mm

Commit message: První prototyp pcb
Parts:
- RX: renamed from UART TX
- moved S2 50.0 mm to (158.6, 134.0), turned to -90 degrees
- moved S3 44.6 mm to (149.3, 134.0), turned to -90 degrees
- moved S4 42.7 mm to (140.0, 134.0), turned to -90 degrees
- moved R3 38.2 mm to (154.0, 127.0), turned to 0 degrees
- moved R2 33.5 mm to (145.0, 127.0), turned to 0 degrees
- moved R1 33.3 mm to (136.0, 127.0), turned to 0 degrees
- moved RX 26.6 mm to (143.0, 107.2), turned to 90 degrees
- moved BZ1 17.0 mm to (168.0, 90.0), turned to 0 degrees
- moved R9 8.67 mm to (114.0, 79.7)
- moved CAMERA 8.67 mm to (117.5, 79.0)
- moved C18 5.66 mm to (133.8, 88.4)
- moved R10 2.93 mm to (121.5, 74.4), turned to 0 degrees
- moved LCD 2.74 mm to (104.6, 86.8)
- moved R13 2.74 mm to (96.0, 88.6)
- moved R8 2.74 mm to (104.0, 97.6)
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Routing:
- net +3.3V: track 18.3 -> 355.6 mm, vias 0 -> 25
- net +3.3V LCD: track 0.00 -> 170.2 mm, vias 0 -> 6
- net /sd miso: track 0.00 -> 142.7 mm, vias 0 -> 4
- net GND: track 54.4 -> 187.3 mm, vias 16 -> 37
- net /scl: track 0.00 -> 128.9 mm, vias 0 -> 10
- net /d3: track 0.00 -> 106.8 mm, vias 0 -> 6
- net /d1: track 0.00 -> 101.5 mm, vias 0 -> 6
- net /d0: track 0.00 -> 101.4 mm, vias 0 -> 9
- net /d2: track 0.00 -> 99.5 mm, vias 0 -> 11
- net /wrx d/cx: track 0.00 -> 96.9 mm, vias 0 -> 4
- net /d6: track 0.00 -> 96.7 mm, vias 0 -> 4
- net /d7: track 0.00 -> 88.6 mm, vias 0 -> 4
- net /d5: track 0.00 -> 87.9 mm, vias 0 -> 4
- net /vsync: track 0.00 -> 87.1 mm, vias 0 -> 4
- net /I2C_SDA: track 0.00 -> 83.6 mm, vias 0 -> 8
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Other:
- board text added: "clk"
- board text added: "io"
